Commit message: Modififed action server to use joint states instead of finger position (for better MoveIt control) and added new collision model with padding

File: robotiq_arg2f_model_visualization/urdf/robotiq_arg2f_140_model_macro.xacro (robot description, xacro)
@@ -27,5 +27,5 @@
         <origin xyz="0 0 0" rpy="0 0 0" />
         <geometry>
-          <mesh filename="package://robotiq_arg2f_model_visualization/meshes/robotiq_arg2f_${stroke}_outer_knuckle.stl" />
+          <mesh filename="package://robotiq_arg2f_model_visualization/meshes/robotiq_arg2f_${stroke}_outer_knuckle_padded.stl" />
         </geometry>
       </collision>
@@ -117,5 +117,5 @@
         <origin xyz="0 0 0" rpy="0 0 0" />
         <geometry>
-          <mesh filename="package://robotiq_arg2f_model_visualization/meshes/robotiq_arg2f_${stroke}_inner_finger.stl" />
+          <mesh filename="package://robotiq_arg2f_model_visualization/meshes/robotiq_arg2f_${stroke}_inner_finger_padded.stl" />
         </geometry>
       </collision>
@@ -136,5 +136,5 @@
       <child link="${prefix}${fingerprefix}_inner_knuckle" />
       <axis xyz="1 0 0" />
-      <limit lower="0" upper="0.8757" velocity="2.0" effort="1000" />
+      <limit lower="-0.8757" upper="0.8757" velocity="2.0" effort="1000" />
       <mimic joint="${prefix}finger_joint" multiplier="-1" offset="0" />
     </joint>
@@ -167,5 +167,5 @@
       <child link="${prefix}right_outer_knuckle" />
       <axis xyz="1 0 0" />
-      <limit lower="0" upper="0.725" velocity="2.0" effort="1000" />
+      <limit lower="-0725" upper="0.725" velocity="2.0" effort="1000" />
     <mimic joint="${prefix}finger_joint" multiplier="-1" offset="0" />
     </joint>
